File: blinking_heart_pcb_keychain/blinking_heart_pcb_keychain.kicad_sch (KiCad schematic)
At the start: 32 parts, among them U1 NE555, U2 CD4017BE

Commit message: Completing most of the routing
Parts:
- added B3: (no value), blinking_heart_pcb_keychain_footprints:MX1A-E1NW, symbol blinking_heart_pcb_keychain_components:MX1A-E1NW
Connections:
- net at D11.2: now also B3.2; no longer B2.1 (+3V)
- new net: B2.1 (+3V), B3.1
Other:
- moved on the sheet: D11
Changed lines of the file:
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@@
 	)
 	(junction
+		(at 82.55 67.31)
+		(diameter 0)
+		(color 0 0 0 0)
+	)
+	(junction
 		(at 245.11 91.44)
 		(diameter 0)
@@
 	)
 	(junction
-		(at 82.55 67.31)
-		(diameter 0)
-		(color 0 0 0 0)
-	)
-	(junction
 		(at 245.11 72.39)
 		(diameter 0)
@@
 	(wire
 		(pts
-			(xy 77.47 67.31) (xy 82.55 67.31)
-		)
-		(stroke
-			(width 0)
-			(type default)
-		)
-	)
-	(wire
-		(pts
 			(xy 96.52 130.81) (xy 99.06 130.81)
 		)
@@
 	(wire
 		(pts
+			(xy 82.55 67.31) (xy 91.44 67.31)
+		)
+		(stroke
+			(width 0)
+			(type default)
+		)
+	)
+	(wire
+		(pts
 			(xy 201.93 87.63) (xy 201.93 78.74)
 		)
@@
 	(wire
 		(pts
-			(xy 160.02 107.95) (xy 154.94 107.95)
+			(xy 81.28 67.31) (xy 82.55 67.31)
 		)
 		(stroke
@@
 	(wire
 		(pts
-			(xy 64.77 67.31) (xy 69.85 67.31)
+			(xy 160.02 107.95) (xy 154.94 107.95)
 		)
 		(stroke
@@
 	(wire
 		(pts
+			(xy 73.66 67.31) (xy 74.93 67.31)
+		)
+		(stroke
+			(width 0)
+			(type default)
+		)
+	)
+	(wire
+		(pts
 			(xy 219.71 91.44) (xy 227.33 91.44)
 		)
@@
 	(wire
 		(pts
-			(xy 82.55 67.31) (xy 91.44 67.31)
+			(xy 96.52 137.16) (xy 96.52 134.62)
 		)
 		(stroke
@@
 	(wire
 		(pts
-			(xy 96.52 137.16) (xy 96.52 134.62)
+			(xy 82.55 78.74) (xy 82.55 81.28)
 		)
 		(stroke
@@
 	(wire
 		(pts
-			(xy 82.55 78.74) (xy 82.55 81.28)
+			(xy 219.71 66.04) (xy 227.33 66.04)
 		)
 		(stroke
@@
 	(wire
 		(pts
-			(xy 219.71 66.04) (xy 227.33 66.04)
+			(xy 82.55 81.28) (xy 88.9 81.28)
 		)
 		(stroke
@@
 	(wire
 		(pts
-			(xy 82.55 81.28) (xy 88.9 81.28)
+			(xy 64.77 67.31) (xy 66.04 67.31)
 		)
 		(stroke
@@
 	(symbol
 		(lib_id "blinking_heart_pcb_keychain_components:D")
-		(at 73.66 67.31 180)
+		(at 78.74 67.31 180)
 		(unit 1)
 		(body_style 1)
@@
 		(fields_autoplaced yes)
 		(property "Reference" "D11"
-			(at 73.66 63.5 0)
+			(at 78.74 63.5 0)
 			(show_name no)
 			(do_not_autoplace no)
@@
 		)
 		(property "Value" ""
-			(at 73.66 67.31 0)
+			(at 78.74 67.31 0)
 			(hide yes)
 			(show_name no)
@@
 		)
 		(property "Footprint" "blinking_heart_pcb_keychain_footprints:D_1N5817"
-			(at 73.66 67.31 0)
+			(at 78.74 67.31 0)
 			(hide yes)
 			(show_name no)
@@
 		)
 		(property "Datasheet" "kicad-embed://1N5817 THRU 1N5819 N0014 REV.C.pdf"
-			(at 73.66 67.31 0)
+			(at 78.74 67.31 0)
 			(hide yes)
 			(show_name no)
@@
 		)
 		(property "Description" "Diode"
-			(at 73.66 67.31 0)
+			(at 78.74 67.31 0)
 			(hide yes)
 			(show_name no)
@@
 		)
 		(property "Digikey" "https://www.digikey.ca/short/b2mjpf39"
-			(at 73.66 67.31 0)
+			(at 78.74 67.31 0)
 			(hide yes)
 			(show_name no)
@@
 					(unit 1)
 				)
+			)
+		)
+	)
+	(symbol
+		(lib_id "blinking_heart_pcb_keychain_components:MX1A-E1NW")
+		(at 69.85 67.31 0)
+		(unit 1)
+		(body_style 1)
+		(exclude_from_sim no)
+		(in_bom yes)
+		(on_board yes)
+		(in_pos_files yes)
+		(dnp no)
+		(fields_autoplaced yes)
+		(property "Reference" "B3"
+			(at 69.85 63.5 0)
+			(show_name no)
+			(do_not_autoplace no)
+			(effects
+				(font
+					(size 1.27 1.27)
+				)
+			)
+		)
+		(property "Value" ""
+			(at 69.85 67.31 0)
+			(show_name no)
+			(do_not_autoplace no)
+			(effects
+				(font
+					(size 1.27 1.27)
+				)
+			)
+		)
+		(property "Footprint" "blinking_heart_pcb_keychain_footprints:MX1A-E1NW"
+			(at 69.85 67.31 0)
+			(hide yes)
+			(show_name no)
+			(do_not_autoplace no)
+			(effects
+				(font
+					(size 1.27 1.27)
+				)
+			)
+		)
+		(property "Datasheet" ""
+			(at 69.85 67.31 0)
+			(hide yes)
+			(show_name no)
+			(do_not_autoplace no)
+			(effects
+				(font
+					(size 1.27 1.27)
+				)
+			)
+		)
+		(property "Description" "SWITCH PUSH SPST-NO 0.01A 12V"
+			(at 69.85 67.31 0)
+			(hide yes)
+			(show_name no)
+			(do_not_autoplace no)
+			(effects
+				(font
+					(size 1.27 1.27)
+				)
+			)
+		)
+		(property "Digikey" "https://www.digikey.ca/short/5j9mnhmb"
+			(at 69.85 67.31 0)
+			(hide yes)
+			(show_name no)
+			(do_not_autoplace no)
+			(effects
+				(font
+					(size 1.27 1.27)
+				)
+			)
+		)
+		(pin "1"
+		)
+		(pin "2"
+		)
+		(instances
+			(project "blinking_heart_pcb_keychain"
+				(path "/7fd9d1ba-6206-442e-99ea-807d70620cf4"
+					(reference "B3")
+					(unit 1)
+				)
