File: blinking_heart_pcb_keychain/blinking_heart_pcb_keychain.kicad_pcb (KiCad board)
At the start: 2 copper layers, 55 x 55 mm, 36 parts, among them U1 NE555, U2 CD4017BE

Commit message: Begining component placement
Parts:
- VR1: moved to B.Cu
- moved U1 81.8 mm to (164.0, 55.5), turned to 180 degrees
- moved C2 71.6 mm to (171.0, 54.5), turned to 90 degrees
- moved U2 71.6 mm to (165.2, 98.1), turned to 180 degrees
- moved C3 70.4 mm to (171.0, 77.5), turned to -90 degrees
- moved VR1 51.4 mm to (151.0, 82.6), turned to 90 degrees
- moved D11 51.1 mm to (175.0, 77.5), turned to -90 degrees
- moved C1 46.2 mm to (275.2, 123.9)
- moved C4 46.2 mm to (275.2, 134.1)
- moved R5 46.2 mm to (267.0, 116.8)
- moved R10 46.2 mm to (267.0, 130.8)
- moved R11 46.2 mm to (267.0, 133.6)
- moved R3 46.2 mm to (267.0, 111.2)
- moved R4 46.2 mm to (267.0, 114.0)
- moved R6 46.2 mm to (267.0, 119.6)
- moved R7 46.2 mm to (267.0, 122.4)
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Other:
- board size 55 x 55 mm -> 100 x 55 mm

Commit message: Completing most of the routing
Parts:
- removed REF** (x4): MountingHole_3.2mm_M3, MountingHole:MountingHole_3.2mm_M3
- added ?: , , F.Cu at (114.4, 125.6)
- added ?: , , F.Cu at (114.4, 49.4)
- added ?: , , F.Cu at (180.6, 125.6)
- added ?: , , F.Cu at (180.6, 49.4)
- added B3: ~, blinking_heart_pcb_keychain_footprints:MX1A-E1NW, F.Cu at (150.0, 117.2)
- VR1: moved to F.Cu
- moved R7 144.0 mm to (135.0, 65.0), turned to 180 degrees
- moved R6 142.1 mm to (135.0, 67.0), turned to 180 degrees
- moved R11 128.4 mm to (148.0, 85.5)
- moved C4 127.7 mm to (160.0, 79.0)
- moved R12 127.2 mm to (148.0, 91.5)
- moved R10 125.6 mm to (159.5, 66.0)
- moved R9 125.1 mm to (159.5, 64.0)
- moved R5 122.6 mm to (148.0, 87.5), turned to 180 degrees
- moved R8 121.8 mm to (159.5, 68.0), turned to 180 degrees
- moved R4 121.5 mm to (148.0, 89.5), turned to 180 degrees
- moved R3 120.3 mm to (148.0, 93.5), turned to 180 degrees
- moved C1 96.8 mm to (182.5, 96.0), turned to -90 degrees
- moved B1 74.3 mm to (130.0, 116.5), turned to 90 degrees
- moved D7 55.1 mm to (160.7, 55.7), turned to 180 degrees
- moved D8 54.9 mm to (170.7, 65.7), turned to 0 degrees
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Connections:
- D11 pad 2: Net-(B2-+3V) -> Net-(B3-Pad2)
Routing:
- net GND: track 0.00 -> 192.7 mm, vias 0 -> 2
- net Net-(U2-OUT_8): track 0.00 -> 113.5 mm, vias 0 -> 2
- net Net-(U2-OUT_6): track 0.00 -> 79.0 mm, vias 0 -> 1
- net Net-(U2-OUT_7): track 0.00 -> 76.6 mm, vias 0 -> 1
- net Net-(B1-+3V): track 0.00 -> 72.5 mm
- net Net-(U2-OUT_9): track 0.00 -> 70.0 mm, vias 0 -> 2
- net Net-(U2-OUT_4): track 0.00 -> 62.1 mm, vias 0 -> 1
- net /CLK: track 0.00 -> 56.4 mm
- net Net-(B2-+3V): track 0.00 -> 52.2 mm, vias 0 -> 1
- net +5V: track 0.00 -> 52.2 mm, vias 0 -> 1
- net Net-(VR1-VIN): track 0.00 -> 40.3 mm, vias 0 -> 1
- net Net-(U2-OUT_5): track 0.00 -> 39.7 mm, vias 0 -> 1
- net Net-(U2-OUT_3): track 0.00 -> 33.1 mm, vias 0 -> 1
- net Net-(U2-OUT_0): track 0.00 -> 30.5 mm
- net Net-(U1-THRES): track 0.00 -> 25.0 mm, vias 0 -> 1
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Other:
- board size 100 x 55 mm -> 75 x 85 mm

Commit message: Setting up all manufacturing files
Routing:
- net +5V: track 52.2 -> 95.2 mm
- net GND: track 192.7 -> 210.0 mm
